Commit message: Add an alternate robot (similar to prev) with an extra mid body coming up from the rectangular chassis
Tested that it is stable and catches the ball

File: task2/workspace/catkin_ws/src/my_robot/urdf/my_robot1.xacro (robot description, xacro)
@@ -7,33 +7,4 @@
     <parent link="robot_footprint"/>
     <child link="chassis" />
-  </joint>
-  <link name='mid_body'>
-      <collision name='mid_body_collision'>
-        <origin xyz="0 0 0" rpy="0 0 0"/>
-        <geometry>
-          <box size=".08 .08 .1"/>
-        </geometry>
-      </collision>
-      <visual name='mid_body_visual'>
-        <origin xyz="0 0 0" rpy="0 0 0"/>
-        <geometry>
-          <box size=".08 .08 .1"/>
-        </geometry>
-      </visual>
-      <inertial>
-        <origin xyz="0 0 0" rpy="0 0 0"/>
-        <mass value="1e-5"/>
-        <inertia
-          ixx="1e-6" ixy="0" ixz="0"
-          iyy="1e-6" iyz="0"
-          izz="1e-6"
-        />
-      </inertial>
-  </link>
-  <joint type="fixed" name="mid_body_hinge">
-    <origin xyz="-0.1 0 0.1" rpy=" 0 0 0"/>
-    <axis xyz="0 1 0"/>
-    <child link="mid_body"/>
-    <parent link="chassis"/>
   </joint>
   <link name='left_wheel'>
