Commit message: Pull the robot closer to main view, and modify R2D2 to standup with a camera !
I am still sticking with the original robot3 robot, as that's a 2 wheel
for which we have the differential drive plugin.

I can continue modifying R2D2 to move by studing its transmission characteristics.

File: task2/workspace/catkin_ws/src/my_robot/urdf/my_robot2.xacro (robot description, xacro)
@@ -1,8 +1,9 @@
 <?xml version="1.0"?>
 <robot name="my_robot" xmlns:xacro="http://ros.org/wiki/xacro">
+<xacro:include filename="$(find my_robot)/urdf/my_robot.gazebo" />
   <xacro:property name="width" value="0.2" />
-  <xacro:property name="leglen" value="0.6" />
+  <xacro:property name="leglen" value="0.5" />
   <xacro:property name="polelen" value="0.2" />
-  <xacro:property name="bodylen" value="0.6" />
+  <xacro:property name="bodylen" value="0.5" />
   <xacro:property name="baselen" value="0.4" />
   <xacro:property name="wheeldiam" value="0.07" />
@@ -37,4 +38,36 @@
     <xacro:default_inertial mass="10"/>
   </link>
+  <link name='camera'>
+    <collision name='cam_collision'>
+      <origin xyz="0 0 0" rpy="0 0 0"/>
+      <geometry>
+        <box size=".05 .05 .05"/>
+      </geometry>
+    </collision>
+    <visual name='cam_visual'>
+      <origin xyz="0 0 0" rpy="0 0 0"/>
+      <geometry>
+        <box size=".05 .05 .05"/>
+      </geometry>
+    </visual>
+    <inertial>
+      <origin xyz="0 0 0" rpy="0 0 0"/>
+      <mass value="0.1"/>
+      <inertia
+        ixx="1e-6" ixy="0" ixz="0"
+        iyy="1e-6" iyz="0"
+        izz="1e-6"
+      />
+    </inertial>
+    <box_inertia sizeX="0.05" sizeY="0.05" sizeZ="0.05" mass="0.1">
+      <origin xyz="0 0 0" rpy="0 0 0" />
+    </box_inertia>
+  </link>
+  <joint type='fixed' name='camera_joint'>
+    <origin xyz="0.2 0 0" rpy=" 0 0 0"/>
+    <axis xyz="0 1 0"/>
+    <child link="camera"/>
+    <parent link="base_link"/>
+  </joint>
   <xacro:macro name="wheel" params="prefix suffix reflect">
     <link name="${prefix}_${suffix}_wheel">
