Commit message: Add left wheel to robot per specifications (urdf)
roslaunch reports a launch error:

[INFO] [1555107709.991239, 0.114000]: Calling service /gazebo/spawn_urdf_model
Error [parser_urdf.cc:3474] Unable to call parseURDF on robot model
Error [parser.cc:341] parse as old deprecated model file failed.

To be debugged..

File: task2/workspace/catkin_ws/src/my_robot/urdf/my_robot.xacro (robot description, xacro)
@@ -6,4 +6,58 @@
     <parent link="robot_footprint"/>
     <child link="chassis" />
+  </joint>
+  <link name='left_wheel'>
+      <collision name='lw_collision'>
+        <origin xyz="0 0 0" rpy="0 1.5707 1.5707"/>
+        <geometry>
+          <cylinder radius="0.1" length="0.05"/>
+        </geometry>
+      </collision>
+      <visual name='lw_visual'>
+        <origin xyz="0 0 0" rpy="0 1.5707 1.5707"/>
+        <geometry>
+          <cylinder radius="0.1" length="0.05"/>
+        </geometry>
+      </visual>
+      <inertial>
+        <origin xyz="0 0 0" rpy="0 1.5707 1.5707"/>
+        <mass value="5"/>
+        <inertia
+          ixx="0.1" ixy="0" ixz="0"
+          iyy="0.1" iyz="0"
+          izz="0.1"
+        />
+      </inertial>
+  </link>
+  <link name='right_wheel'>
+      <collision name='rw_collision'>
+        <origin xyz="0 0 0" rpy="0 1.5707 1.5707"/>
+        <geometry>
+          <cylinder radius="0.1" length="0.05"/>
+        </geometry>
+      </collision>
+      <visual name='rw_visual'>
+        <origin xyz="0 0 0" rpy="0 1.5707 1.5707"/>
+        <geometry>
+          <cylinder radius="0.1" length="0.05"/>
+        </geometry>
+      </visual>
+      <inertial>
+        <origin xyz="0 0 0" rpy="0 1.5707 1.5707"/>
+        <mass value="5"/>
+        <inertia
+          ixx="0.1" ixy="0" ixz="0"
+          iyy="0.1" iyz="0"
+          izz="0.1"
+        />
+      </inertial>
+  </link>
+  <joint type="continuous" name="left_wheel_hinge">
+    <origin xyz="0 0.15 0" rpy="0 0 0"/>
+    <child link="left_wheel"/>
+    <parent link="chassis"/>
+    <axis xyz="0 1 0" rpy="0 0 0"/>
+    <limit effort="10000" velocity="1000"/>
+    <dynamics damping="1.0" friction="1.0"/>
   </joint>
   <link name='chassis'>

Commit message: Fixed urdf parser error - deleted unassociated right wheel link
Looks like parser actually structurally tries to construct and blanks
out when it fails. I had just added the right wheel link without its
corresponding joint to the robot chassis ... hmm, good to know..?

File: task2/workspace/catkin_ws/src/my_robot/urdf/my_robot.xacro (robot description, xacro)
@@ -15,27 +15,4 @@
       </collision>
       <visual name='lw_visual'>
-        <origin xyz="0 0 0" rpy="0 1.5707 1.5707"/>
-        <geometry>
-          <cylinder radius="0.1" length="0.05"/>
-        </geometry>
-      </visual>
-      <inertial>
-        <origin xyz="0 0 0" rpy="0 1.5707 1.5707"/>
-        <mass value="5"/>
-        <inertia
-          ixx="0.1" ixy="0" ixz="0"
-          iyy="0.1" iyz="0"
-          izz="0.1"
-        />
-      </inertial>
-  </link>
-  <link name='right_wheel'>
-      <collision name='rw_collision'>
-        <origin xyz="0 0 0" rpy="0 1.5707 1.5707"/>
-        <geometry>
-          <cylinder radius="0.1" length="0.05"/>
-        </geometry>
-      </collision>
-      <visual name='rw_visual'>
         <origin xyz="0 0 0" rpy="0 1.5707 1.5707"/>
         <geometry>

Commit message: Add the right wheel and joint, and it works
Used the left wheel as template. All I had to do was
to modify the y value of the joint to a negative mirror (-0.15)

File: task2/workspace/catkin_ws/src/my_robot/urdf/my_robot.xacro (robot description, xacro)
@@ -33,4 +33,35 @@
     <origin xyz="0 0.15 0" rpy="0 0 0"/>
     <child link="left_wheel"/>
+    <parent link="chassis"/>
+    <axis xyz="0 1 0" rpy="0 0 0"/>
+    <limit effort="10000" velocity="1000"/>
+    <dynamics damping="1.0" friction="1.0"/>
+  </joint>
+  <link name='right_wheel'>
+      <collision name='rw_collision'>
+        <origin xyz="0 0 0" rpy="0 1.5707 1.5707"/>
+        <geometry>
+          <cylinder radius="0.1" length="0.05"/>
+        </geometry>
+      </collision>
+      <visual name='rw_visual'>
+        <origin xyz="0 0 0" rpy="0 1.5707 1.5707"/>
+        <geometry>
+          <cylinder radius="0.1" length="0.05"/>
+        </geometry>
+      </visual>
+      <inertial>
+        <origin xyz="0 0 0" rpy="0 1.5707 1.5707"/>
+        <mass value="5"/>
+        <inertia
+          ixx="0.1" ixy="0" ixz="0"
+          iyy="0.1" iyz="0"
+          izz="0.1"
+        />
+      </inertial>
+  </link>
+  <joint type="continuous" name="right_wheel_hinge">
+    <origin xyz="0 -0.15 0" rpy="0 0 0"/>
+    <child link="right_wheel"/>
     <parent link="chassis"/>
     <axis xyz="0 1 0" rpy="0 0 0"/>

Commit message: Add camera link and joint
But I dont see it displayed, neither do I see gazebo show the link
in the object descriptor ..

File: task2/workspace/catkin_ws/src/my_robot/urdf/my_robot.xacro (robot description, xacro)
@@ -69,4 +69,33 @@
     <dynamics damping="1.0" friction="1.0"/>
   </joint>
+  <link name='camera'>
+    <collision name='cam_collision'>
+      <origin xyz="0 0 0" rpy="0 0 0"/>
+      <geometry>
+        <box size="0.05 0.05 0.05"/>
+      </geometry>
+    </collision>
+    <visual name='cam_visual'>
+      <origin xyz="0 0 0" rpy="0 0 0"/>
+      <geometry>
+        <box size="0.05 0.05 0.05"/>
+      </geometry>
+    </visual>
+    <inertial>
+      <origin xyz="0 0 0" rpy="0 0 0"/>
+      <mass value="0.1"/>
+      <inertia
+        ixx="1e-6" ixy="0" ixz="0"
+        iyy="1e-6" iyz="0"
+        izz="1e-6"
+      />
+    </inertial>
+  </link>
+  <joint name='camera_joint' type='fixed'>
+    <origin xyz="0.2 0 0" rpy=" 0 0 0"/>
+    <axis xyz="0 1 0"/>
+    <child link="camera"/>
+    <parent link="chassis"/>
+  </joint>
   <link name='chassis'>
     <pose>0 0 0.1 0 0 0</pose>

Commit message: Add material color and box_inertial but still no visible camera
checked that my_robot.xacro is correct by removing a wheel.
bizzare!

File: task2/workspace/catkin_ws/src/my_robot/urdf/my_robot.xacro (robot description, xacro)
@@ -19,4 +19,7 @@
           <cylinder radius="0.1" length="0.05"/>
         </geometry>
+        <material name='blue'>
+            <color rgba="0 0 .8 1"/>
+        </material>
       </visual>
       <inertial>
@@ -108,4 +111,7 @@
           izz="0.1"
       />
+      <box_inertia>
+        <mass value="0.1" xyz="0.05 0.05 0.05"/>
+      </box_inertia>
     </inertial>
     <collision name='collision'>

Commit message: Camera is visible
Added a few cosmetic changes. Color still doesn't show
Put box_inertia to camera (instea of chassis)
Maybe the camera box was always showing .. didn't check.

File: task2/workspace/catkin_ws/src/my_robot/urdf/my_robot.xacro (robot description, xacro)
@@ -76,5 +76,5 @@
       <origin xyz="0 0 0" rpy="0 0 0"/>
       <geometry>
-        <box size="0.05 0.05 0.05"/>
+        <box size=".05 .05 .05"/>
       </geometry>
     </collision>
@@ -82,6 +82,9 @@
       <origin xyz="0 0 0" rpy="0 0 0"/>
       <geometry>
-        <box size="0.05 0.05 0.05"/>
+        <box size=".05 .05 .05"/>
       </geometry>
+      <material name='blue'>
+          <color rgba="0 0 .8 1"/>
+      </material>
     </visual>
     <inertial>
@@ -94,6 +97,9 @@
       />
     </inertial>
+    <box_inertia sizeX="0.05" sizeY="0.05" sizeZ="0.05" mass="0.1">
+      <origin xyz="0 0 0" rpy="0 0 0" />
+    </box_inertia>
   </link>
-  <joint name='camera_joint' type='fixed'>
+  <joint type='fixed' name='camera_joint'>
     <origin xyz="0.2 0 0" rpy=" 0 0 0"/>
     <axis xyz="0 1 0"/>
@@ -111,7 +117,4 @@
           izz="0.1"
       />
-      <box_inertia>
-        <mass value="0.1" xyz="0.05 0.05 0.05"/>
-      </box_inertia>
     </inertial>
     <collision name='collision'>

Commit message: Add Hokuyo Lidar sensor
Checked that it is visually added to robot

File: task2/workspace/catkin_ws/src/my_robot/urdf/my_robot.xacro (robot description, xacro)
@@ -107,4 +107,35 @@
     <parent link="chassis"/>
   </joint>
+  <link name='hokuyo'>
+    <collision name='lidar_collision'>
+      <origin xyz="0 0 0" rpy="0 0 0"/>
+      <geometry>
+        <box
+          size="0.1 0.1 0.1"
+        />
+      </geometry>
+    </collision>
+    <visual name='lidar_visual'>
+      <origin xyz="0 0 0" rpy="0 0 0"/>
+      <geometry>
+        <mesh filename="package://my_robot/meshes/hokuyo.dae"/>
+      </geometry>
+    </visual>
+    <inertial>
+      <origin xyz="0 0 0" rpy="0 0 0"/>
+      <mass value="1e-5"/>
+      <inertia
+        ixx="1e-6" ixy="0" ixz="0"
+        iyy="1e-6" iyz="0"
+        izz="1e-6"
+      />
+    </inertial>
+  </link>
+  <joint type='fixed' name='hokuyo_joint'>
+    <origin xyz="0.15 0 0.1" rpy=" 0 0 0"/>
+    <axis xyz="0 1 0"/>
+    <child link="hokuyo"/>
+    <parent link="chassis"/>
+  </joint>
   <link name='chassis'>
     <pose>0 0 0.1 0 0 0</pose>

Commit message: Make chassis a square instead of rect
Also add a second .xacro robot model that more resembles an R2D2 shape ..

Checked that with the squared chassis, my robot still chases the ball.
Only thing is that its not in view now, so jump to top view to make it work.

Can also save the world file with the correct orientation, but not now ..

File: task2/workspace/catkin_ws/src/my_robot/urdf/my_robot.xacro (robot description, xacro)
@@ -20,7 +20,4 @@
           <cylinder radius="0.1" length="0.05"/>
         </geometry>
-        <material name='blue'>
-            <color rgba="0 1 1 1"/>
-        </material>
       </visual>
       <inertial>
@@ -85,7 +82,4 @@
         <box size=".05 .05 .05"/>
       </geometry>
-      <material name='blue'>
-          <color rgba="0 0 .8 1"/>
-      </material>
     </visual>
     <inertial>
@@ -153,5 +147,5 @@
       <origin xyz="0 0 0" rpy=" 0 0 0"/>
       <geometry>
-        <box size=".4 .2 .1"/>
+        <box size=".4 .4 .1"/>
       </geometry>
     </collision>
@@ -159,6 +153,9 @@
       <origin xyz="0 0 0" rpy=" 0 0 0"/>
       <geometry>
-        <box size=".4 .2 .1"/>
+        <box size=".4 .4 .1"/>
       </geometry>
+      <material name="Cyan">
+        <color rgba="0 1.0 1.0 1.0"/>
+      </material>
     </visual>
     <collision name='back_caster_collision'>

Commit message: Cosmetics: Align the wheels a little more outward ..

File: task2/workspace/catkin_ws/src/my_robot/urdf/my_robot.xacro (robot description, xacro)
@@ -61,5 +61,5 @@
   </link>
   <joint type="continuous" name="left_wheel_hinge">
-    <origin xyz="0 0.15 0" rpy="0 0 0"/>
+    <origin xyz="0 0.2 0" rpy="0 0 0"/>
     <child link="left_wheel"/>
     <parent link="chassis"/>
@@ -92,5 +92,5 @@
   </link>
   <joint type="continuous" name="right_wheel_hinge">
-    <origin xyz="0 -0.15 0" rpy="0 0 0"/>
+    <origin xyz="0 -0.2 0" rpy="0 0 0"/>
     <child link="right_wheel"/>
     <parent link="chassis"/>

Commit message: Add gazbo tag for color to robot
Still camera, wheels and casters don't color. Don't know why.
Moving on..

File: task2/workspace/catkin_ws/src/my_robot/urdf/my_robot.xacro (robot description, xacro)
@@ -162,4 +162,25 @@
     <parent link="chassis"/>
   </joint>
+  <gazebo reference="chassis">
+    <material> Gazebo/Orange</material>">
+  </gazebo>
+  <gazebo reference="camera">
+    <material> Gazebo/Red</material>">
+  </gazebo>
+  <gazebo reference="left_wheel">
+    <material> Gazebo/Green</material>">
+  </gazebo>
+  <gazebo reference="right_wheel">
+    <material> Gazebo/Green</material>">
+  </gazebo>
+  <gazebo reference="mid_body">
+    <material> Gazebo/Turquoise</material>">
+  </gazebo>
+  <gazebo reference="chassis/back_caster_visual">
+    <material> Gazebo/Yellow</material>">
+  </gazebo>
+  <gazebo reference="chassis/front_caster_visual">
+    <material> Gazebo/Yellow</material>">
+  </gazebo>
   <link name='chassis'>
     <pose>0 0 0.1 0 0 0</pose>
@@ -184,7 +205,4 @@
         <box size=".4 .4 .1"/>
       </geometry>
-      <material name="Cyan">
-        <color rgba="0 1.0 1.0 1.0"/>
-      </material>
     </visual>
     <collision name='back_caster_collision'>

Commit message: Fix colors for wheels and camera
This was fixed by using the parent link name as prefix for the respective visual.

It doesn't address the problem of coloring multiple visuals inside a link
(e.g. the sphere geometries for the caster visuals, which still do not acquire color)

File: task2/workspace/catkin_ws/src/my_robot/urdf/my_robot.xacro (robot description, xacro)
@@ -38,5 +38,5 @@
   </joint>
   <link name='left_wheel'>
-      <collision name='lw_collision'>
+      <collision name='left_wheel_collision'>
         <origin xyz="0 0 0" rpy="0 1.5707 1.5707"/>
         <geometry>
@@ -44,5 +44,5 @@
         </geometry>
       </collision>
-      <visual name='lw_visual'>
+      <visual name='left_wheel_visual'>
         <origin xyz="0 0 0" rpy="0 1.5707 1.5707"/>
         <geometry>
@@ -69,5 +69,5 @@
   </joint>
   <link name='right_wheel'>
-      <collision name='rw_collision'>
+      <collision name='right_wheel_collision'>
         <origin xyz="0 0 0" rpy="0 1.5707 1.5707"/>
         <geometry>
@@ -75,5 +75,5 @@
         </geometry>
       </collision>
-      <visual name='rw_visual'>
+      <visual name='right_wheel_visual'>
         <origin xyz="0 0 0" rpy="0 1.5707 1.5707"/>
         <geometry>
@@ -100,5 +100,5 @@
   </joint>
   <link name='camera'>
-    <collision name='cam_collision'>
+    <collision name='camera_collision'>
       <origin xyz="0 0 0" rpy="0 0 0"/>
       <geometry>
@@ -106,5 +106,5 @@
       </geometry>
     </collision>
-    <visual name='cam_visual'>
+    <visual name='camera_visual'>
       <origin xyz="0 0 0" rpy="0 0 0"/>
       <geometry>
@@ -163,23 +163,23 @@
   </joint>
   <gazebo reference="chassis">
-    <material> Gazebo/Orange</material>">
+    <material> Gazebo/Orange</material>
   </gazebo>
   <gazebo reference="camera">
-    <material> Gazebo/Red</material>">
+    <material> Gazebo/Red</material>
   </gazebo>
   <gazebo reference="left_wheel">
-    <material> Gazebo/Green</material>">
+    <material> Gazebo/Yellow</material>
   </gazebo>
   <gazebo reference="right_wheel">
-    <material> Gazebo/Green</material>">
+    <material> Gazebo/Yellow</material>
   </gazebo>
   <gazebo reference="mid_body">
-    <material> Gazebo/Turquoise</material>">
-  </gazebo>
-  <gazebo reference="chassis/back_caster_visual">
-    <material> Gazebo/Yellow</material>">
-  </gazebo>
-  <gazebo reference="chassis/front_caster_visual">
-    <material> Gazebo/Yellow</material>">
+    <material> Gazebo/Turquoise</material>
+  </gazebo>
+  <gazebo reference="back_caster_visual">
+    <material> Gazebo/Green</material>
+  </gazebo>
+  <gazebo reference="front_caster_visual">
+    <material> Gazebo/Green</material>
   </gazebo>
   <link name='chassis'>
@@ -194,5 +194,5 @@
       />
     </inertial>
-    <collision name='collision'>
+    <collision name='chassis_collision'>
       <origin xyz="0 0 0" rpy=" 0 0 0"/>
       <geometry>
