Commit message: sensor upgrade: add rgbd camera code
- haven't removed the old camera yet but added code for new one
- made sure the joint points to the old camera link. checked that it works
- can still see rgb/raw_image (and added that to task4's amcl.rviz)
- changed robot's camera from red to blue (just to visually indicate some difference)
- task2: doesn't load up sensor.rviz (even after calling find_package) .. needs debugging
- cleanup in task4: remove extra .xacro files for my robot, and some unneccesary files

File: task4/workspace/catkin_ws/src/my_robot/urdf/my_robot.xacro (robot description, xacro)
@@ -131,4 +131,11 @@
     <parent link="chassis"/>
   </joint>
+  <joint name="camera_optical_joint" type="fixed">
+    <origin xyz="0 0 0" rpy="-1.5707 0 -1.5707"/>
+    <child link="camera_link_optical"/>
+    <parent link="camera"/>
+  </joint>
+  <link name="camera_link_optical">
+  </link>
   <link name='hokuyo'>
     <collision name='lidar_collision'>
@@ -166,5 +173,5 @@
   </gazebo>
   <gazebo reference="camera">
-    <material> Gazebo/Red</material>
+    <material> Gazebo/Blue</material>
   </gazebo>
   <gazebo reference="left_wheel">
